File: Belja80.kicad_pcb (KiCad board)
At the start: 2 copper layers, 223 parts, among them J1 USB_C_Receptacle_USB2.0, SW1 SW_Esc, SW10 SW_F9, SW11 SW_F10, SW12 SW_F11, SW13 SW_F12, SW14 SW_PrintSc, SW15 SW_ScrollLock, SW16 SW_§, SW17 SW_1, SW18 SW_2, SW19 SW_3, SW2 SW_F1, SW20 SW_4, SW21 SW_6, SW22 SW_7, SW23 SW_8, SW24 SW_0, SW25 SW_+, SW26 SW_|, SW27 SW_Backspace, SW28 SW_Insert, SW29 SW_Home, SW3 SW_F2, SW30 SW_Pause, SW31 SW_Tab, SW32 SW_Q, SW33 SW_W, SW34 SW_E, SW35 SW_R, SW36 SW_5, SW37 SW_Y, SW38 SW_9, SW39 SW_O, SW4 SW_F3, SW40 SW_P, SW41 SW_Å, SW42 SW_^, SW43 SW_Delete, SW44 SW_End, SW45 SW_PgUp, SW46 SW_Caps, SW47 SW_A, SW48 SW_S, SW49 SW_D, SW5 SW_F4, SW50 SW_F, SW51 SW_T, SW52 SW_U, SW53 SW_I, SW54 SW_L, SW55 SW_Æ, SW56 SW_Ø, SW57 SW_*, SW58 SW_\, SW59 SW_ArrowUp, SW6 SW_F5, SW60 SW_PgDn, SW61 SW_LShift2.25u, SW62 SW_EnterISO, SW63 SW_LShift1.25u, SW64 SW_<>, SW65 SW_Z, SW66 SW_X, SW67 SW_C, SW68 SW_G, SW69 SW_H, SW7 SW_F6, SW70 SW_J, SW71 SW_K, SW72 SW_dot, SW73 SW_-, SW74 SW_RShift2.75u, SW75 SW_EnterANSI, SW76 SW_ArrowDown, SW77 SW_ArrowRight, SW78 SW_Ctrl, SW79 SW_Win, SW8 SW_F7, SW80 SW_Alt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

Commit message: Rough layout
Parts:
- C1, C10, C11, C12, C13, C14, C15, C16, C2, C3, C4, C5, C6, C7, C8, C9, D1, D10, D11, D12, D13, D14, D15, D16, D17, D18, D19, D2, D20, D21, D22, D23, D24, D25, D26, D27, D28, D29, D3, D30, D31, D32, D33, D34, D35, D36, D37, D38, D39, D4, D40, D41, D42, D43, D44, D45, D46, D47, D48, D49, D5, D50, D51, D52, D53, D54, D55, D56, D57, D58, D59, D6, D60, D61, D62, D63, D64, D65, D66, D67, D68, D69, D7, D70, D71, D72, D73, D74, D75, D76, D77, D78, D79, D8, D80, D81, D82, D83, D84, D85, D86, D87, D88, D89, D9, D90, F1, FB1, R1, R2, R4, R5, R7, R8, R9, SW92, SW93, U1, U2, U3, Y1: moved to B.Cu
- J1: footprint Belja80:USB_C_Receptacle_GCT_USB4085 -> Connector_USB:USB_C_Receptacle_Palconn_UTC16-G; moved to B.Cu
- R3, R6: footprint Resistor_SMD:R_0603_1608Metric -> Resistor_SMD:R_0402_1005Metric; moved to B.Cu
- moved SW47 624.7 mm to (83.5, 109.2)
- moved SW48 619.5 mm to (102.6, 109.2)
- moved D12 597.6 mm to (187.4, 229.1), turned to 180 degrees
- moved D26 590.0 mm to (192.8, 232.5), turned to 180 degrees
- moved D20 588.7 mm to (192.8, 212.4), turned to 180 degrees
- moved D10 582.6 mm to (187.4, 222.4), turned to 180 degrees
- moved SW35 579.6 mm to (135.9, 90.2)
- moved D19 576.4 mm to (192.8, 209.0), turned to 180 degrees
- moved D31 575.6 mm to (198.3, 205.7), turned to 180 degrees
- moved D54 574.8 mm to (209.3, 195.6), turned to 180 degrees
- moved D65 570.4 mm to (209.3, 232.5), turned to 180 degrees
- moved D1 570.3 mm to (187.4, 192.3), turned to 180 degrees
- moved D66 567.9 mm to (214.8, 192.3), turned to 180 degrees
- moved D77 567.1 mm to (214.8, 229.1), turned to 180 degrees
- moved D61 564.2 mm to (209.3, 219.1), turned to 180 degrees
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Connections:
- C3 pad 1: +3V3 -> /VREG_VOUT
- C4 pad 1: +3V3 -> /VREG_VOUT
- U1 pad 23: +3V3 -> /VREG_VOUT
- U1 pad 50: +3V3 -> /VREG_VOUT
Other:
- board outline added: 347.7 x 126.2 mm
