File: Belja80_plate/Belja80_plate.kicad_pcb (KiCad board)
At the start: 2 copper layers, 347.7 x 126.2 mm, 9 parts

Commit message: Ready for production
Changed lines of the file:
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@@
     (pad_to_mask_clearance 0)
     (pcbplotparams
-      (layerselection 0x00010fc_ffffffff)
+      (layerselection 0x00010c0_ffffffff)
       (plot_on_all_layers_selection 0x0000000_00000000)
       (disableapertmacros false)
-      (usegerberextensions false)
-      (usegerberattributes true)
-      (usegerberadvancedattributes true)
-      (creategerberjobfile true)
+      (usegerberextensions true)
+      (usegerberattributes false)
+      (usegerberadvancedattributes false)
+      (creategerberjobfile false)
       (dashed_line_dash_ratio 12.000000)
       (dashed_line_gap_ratio 3.000000)
@@
       (psa4output false)
       (plotreference true)
-      (plotvalue true)
+      (plotvalue false)
       (plotinvisibletext false)
       (sketchpadsonfab false)
-      (subtractmaskfromsilk false)
+      (subtractmaskfromsilk true)
       (outputformat 1)
       (mirror false)
-      (drillshape 1)
+      (drillshape 0)
       (scaleselection 1)
       (outputdirectory "")
@@
         (effects (font (size 1.27 1.27) (thickness 0.15)))
     )
-    (pad "1" np_thru_hole circle (at 0 0) (size 7 7) (drill 7) (layers "*.Cu" "*.Mask")
+    (pad "" np_thru_hole circle (at 0 0) (size 7 7) (drill 7) (layers "*.Cu" "*.Mask")
       (pinfunction "1") (pintype "input"))
   )
@@
         (effects (font (size 1.27 1.27) (thickness 0.15)))
     )
-    (pad "1" np_thru_hole circle (at 0 0) (size 7 7) (drill 7) (layers "*.Cu" "*.Mask")
+    (pad "" np_thru_hole circle (at 0 0) (size 7 7) (drill 7) (layers "*.Cu" "*.Mask")
       (pinfunction "1") (pintype "input"))
   )
@@
         (effects (font (size 1.27 1.27) (thickness 0.15)))
     )
-    (pad "1" np_thru_hole circle (at 0 0) (size 7 7) (drill 7) (layers "*.Cu" "*.Mask")
+    (pad "" np_thru_hole circle (at 0 0) (size 7 7) (drill 7) (layers "*.Cu" "*.Mask")
       (pinfunction "1") (pintype "input"))
   )
@@
         (effects (font (size 1.27 1.27) (thickness 0.15)))
     )
-    (pad "1" np_thru_hole circle (at 0 0) (size 7 7) (drill 7) (layers "*.Cu" "*.Mask")
+    (pad "" np_thru_hole circle (at 0 0) (size 7 7) (drill 7) (layers "*.Cu" "*.Mask")
       (pinfunction "1") (pintype "input"))
   )
@@
         (effects (font (size 1.27 1.27) (thickness 0.15)))
     )
-    (pad "1" np_thru_hole circle (at 0 0) (size 7 7) (drill 7) (layers "*.Cu" "*.Mask")
+    (pad "" np_thru_hole circle (at 0 0) (size 7 7) (drill 7) (layers "*.Cu" "*.Mask")
       (pinfunction "1") (pintype "input"))
   )
@@
         (effects (font (size 1.27 1.27) (thickness 0.15)))
     )
-    (pad "1" np_thru_hole circle (at 0 0) (size 7 7) (drill 7) (layers "*.Cu" "*.Mask")
+    (pad "" np_thru_hole circle (at 0 0) (size 7 7) (drill 7) (layers "*.Cu" "*.Mask")
       (pinfunction "1") (pintype "input"))
   )
@@
         (effects (font (size 1.27 1.27) (thickness 0.15)))
     )
-    (pad "1" np_thru_hole circle (at 0 0) (size 7 7) (drill 7) (layers "*.Cu" "*.Mask")
+    (pad "" np_thru_hole circle (at 0 0) (size 8 8) (drill 8) (layers "*.Cu" "*.Mask")
       (pinfunction "1") (pintype "input"))
   )
@@
         (effects (font (size 1.27 1.27) (thickness 0.15)))
     )
-    (pad "1" np_thru_hole circle (at 0 0) (size 7 7) (drill 7) (layers "*.Cu" "*.Mask")
+    (pad "" np_thru_hole circle (at 0 0) (size 7 7) (drill 7) (layers "*.Cu" "*.Mask")
       (pinfunction "1") (pintype "input"))
   )
@@
         (effects (font (size 1.27 1.27) (thickness 0.15)))
     )
-    (pad "1" np_thru_hole circle (at 0 0) (size 7 7) (drill 7) (layers "*.Cu" "*.Mask")
+    (pad "" np_thru_hole circle (at 0 0) (size 7 7) (drill 7) (layers "*.Cu" "*.Mask")
       (pinfunction "1") (pintype "input"))
   )
